File: file607D6509.sch (KiCad schematic (older format))
At the start: 15 parts, among them SW1 SW_SPDT, U1 TPS54228DDA

Commit message: full schematic, version 1.0
Parts:
- removed SW1: SW_SPDT, symbol Switch:SW_SPDT
- added S9: EG1218, EIPP:EG1218, symbol EIPP_LIBRARY:EG1218
- C1, C2, C3, C4: footprint (none) -> Capacitor_SMD:C_0603_1608Metric_Pad1.08x0.95mm_HandSolder
- C10, C11: footprint (none) -> Capacitor_SMD:C_1206_3216Metric_Pad1.33x1.80mm_HandSolder
- C5, C8, C9: footprint (none) -> Capacitor_SMD:C_0805_2012Metric_Pad1.18x1.45mm_HandSolder
- L1: value 3u3 -> 3.3uH; footprint (none) -> EIPP:HM66M
- R1, R3: footprint (none) -> Resistor_SMD:R_0805_2012Metric_Pad1.20x1.40mm_HandSolder
- R2: footprint (none) -> Resistor_SMD:R_0603_1608Metric_Pad0.98x0.95mm_HandSolder
- U1: footprint (none) -> EIPP:NOPB
Connections:
- net +BATT: now also S9.S
- net GND: now also S9.O
- net VIN_TPS: now also S9.P
Changed lines of the file:
@@
 $Descr A4 11693 8268
 encoding utf-8
-Sheet 3 10
+Sheet 3 15
 Title ""
 Date ""
@@
 F 0 "U1" H 3425 2615 50  0000 C CNN
 F 1 "TPS54228DDA" H 3425 2524 50  0000 C CNN
-F 2 "" H 3400 2500 50  0001 C CNN
+F 2 "EIPP:NOPB" H 3400 2500 50  0001 C CNN
 F 3 "" H 3400 2500 50  0001 C CNN
 	1    3400 2500
@@
 F 0 "R1" V 1750 2600 50  0000 C CNN
 F 1 "73.2k" V 1900 2600 50  0000 C CNN
-F 2 "" H 1850 2750 50  0001 C CNN
+F 2 "Resistor_SMD:R_0805_2012Metric_Pad1.20x1.40mm_HandSolder" H 1850 2750 50  0001 C CNN
 F 3 "~" H 1850 2750 50  0001 C CNN
 	1    1850 2750
@@
 F 0 "R2" H 2050 3200 50  0000 L CNN
 F 1 "22.1k" H 2059 3055 50  0000 L CNN
-F 2 "" H 2000 3100 50  0001 C CNN
+F 2 "Resistor_SMD:R_0603_1608Metric_Pad0.98x0.95mm_HandSolder" H 2000 3100 50  0001 C CNN
 F 3 "~" H 2000 3100 50  0001 C CNN
 	1    2000 3100
@@
 F 0 "C2" H 2542 3196 50  0000 L CNN
 F 1 "1uF" H 2542 3105 50  0000 L CNN
-F 2 "" H 2450 3150 50  0001 C CNN
+F 2 "Capacitor_SMD:C_0603_1608Metric_Pad1.08x0.95mm_HandSolder" H 2450 3150 50  0001 C CNN
 F 3 "~" H 2450 3150 50  0001 C CNN
 	1    2450 3150
@@
 F 0 "C3" H 2842 3196 50  0000 L CNN
 F 1 "3300pF" H 2842 3105 50  0000 L CNN
-F 2 "" H 2750 3150 50  0001 C CNN
+F 2 "Capacitor_SMD:C_0603_1608Metric_Pad1.08x0.95mm_HandSolder" H 2750 3150 50  0001 C CNN
 F 3 "~" H 2750 3150 50  0001 C CNN
 	1    2750 3150
@@
 U 1 1 607E16DC
 P 4300 2850
-F 0 "L1" V 4400 2850 50  0000 C CNN
-F 1 "3u3" V 4400 2700 50  0000 C CNN
-F 2 "" H 4300 2850 50  0001 C CNN
+F 0 "L1" V 4400 2900 50  0000 C CNN
+F 1 "3.3uH" V 4400 2700 50  0000 C CNN
+F 2 "EIPP:HM66M" H 4300 2850 50  0001 C CNN
 F 3 "~" H 4300 2850 50  0001 C CNN
 	1    4300 2850
@@
 F 0 "C5" H 4400 3200 50  0000 L CNN
 F 1 "22uF" H 4350 3000 50  0000 L CNN
-F 2 "" H 4550 3100 50  0001 C CNN
+F 2 "Capacitor_SMD:C_0805_2012Metric_Pad1.18x1.45mm_HandSolder" H 4550 3100 50  0001 C CNN
 F 3 "~" H 4550 3100 50  0001 C CNN
 	1    4550 3100
@@
 F 0 "C4" V 3900 2800 50  0000 L CNN
 F 1 "0.1uF" V 3800 2850 50  0000 L CNN
-F 2 "" H 3950 2750 50  0001 C CNN
+F 2 "Capacitor_SMD:C_0603_1608Metric_Pad1.08x0.95mm_HandSolder" H 3950 2750 50  0001 C CNN
 F 3 "~" H 3950 2750 50  0001 C CNN
 	1    3950 2750
@@
 F 0 "C1" H 1600 2000 50  0000 L CNN
 F 1 "100nF" H 1450 1850 50  0000 L CNN
-F 2 "" H 1750 1900 50  0001 C CNN
+F 2 "Capacitor_SMD:C_0603_1608Metric_Pad1.08x0.95mm_HandSolder" H 1750 1900 50  0001 C CNN
 F 3 "~" H 1750 1900 50  0001 C CNN
 	1    1750 1900
@@
 F 0 "C8" V 1800 2850 50  0000 C CNN
 F 1 "22p" V 1800 3050 50  0000 C CNN
-F 2 "" H 1750 2950 50  0001 C CNN
+F 2 "Capacitor_SMD:C_0805_2012Metric_Pad1.18x1.45mm_HandSolder" H 1750 2950 50  0001 C CNN
 F 3 "~" H 1750 2950 50  0001 C CNN
 	1    1750 2950
@@
 F 0 "C9" H 4900 3200 50  0000 L CNN
 F 1 "22uF" H 4900 3000 50  0000 L CNN
-F 2 "" H 4850 3100 50  0001 C CNN
+F 2 "Capacitor_SMD:C_0805_2012Metric_Pad1.18x1.45mm_HandSolder" H 4850 3100 50  0001 C CNN
 F 3 "~" H 4850 3100 50  0001 C CNN
 	1    4850 3100
@@
 F 0 "C10" H 1950 2000 50  0000 L CNN
 F 1 "5uF" H 2000 1850 50  0000 L CNN
-F 2 "" H 1950 1900 50  0001 C CNN
+F 2 "Capacitor_SMD:C_1206_3216Metric_Pad1.33x1.80mm_HandSolder" H 1950 1900 50  0001 C CNN
 F 3 "~" H 1950 1900 50  0001 C CNN
 	1    1950 1900
@@
 F 0 "C11" H 2250 2000 50  0000 L CNN
 F 1 "5uF" H 2250 1850 50  0000 L CNN
-F 2 "" H 2200 1900 50  0001 C CNN
+F 2 "Capacitor_SMD:C_1206_3216Metric_Pad1.33x1.80mm_HandSolder" H 2200 1900 50  0001 C CNN
 F 3 "~" H 2200 1900 50  0001 C CNN
 	1    2200 1900
@@
 F 0 "R3" V 2554 2650 50  0000 C CNN
 F 1 "10k" V 2645 2650 50  0000 C CNN
-F 2 "" H 2750 2650 50  0001 C CNN
+F 2 "Resistor_SMD:R_0805_2012Metric_Pad1.20x1.40mm_HandSolder" H 2750 2650 50  0001 C CNN
 F 3 "~" H 2750 2650 50  0001 C CNN
 	1    2750 2650
@@
 $EndComp
 Wire Wire Line
-	4700 1350 5250 1350
-$Comp
-L power:+BATT #PWR09
-U 1 1 6084571D
-P 4700 1350
-F 0 "#PWR09" H 4700 1200 50  0001 C CNN
-F 1 "+BATT" H 4715 1523 50  0000 C CNN
-F 2 "" H 4700 1350 50  0001 C CNN
-F 3 "" H 4700 1350 50  0001 C CNN
-	1    4700 1350
-	1    0    0    -1
-$EndComp
-Wire Wire Line
 	2500 1750 3900 1750
 Wire Wire Line
@@
 Wire Wire Line
 	2500 2650 2500 1750
-$Comp
-L Switch:SW_SPDT SW1
-U 1 1 6084CB97
-P 5450 1450
-F 0 "SW1" H 5450 1125 50  0000 C CNN
-F 1 "SW_SPDT" H 5450 1216 50  0000 C CNN
-F 2 "" H 5450 1450 50  0001 C CNN
-F 3 "~" H 5450 1450 50  0001 C CNN
-	1    5450 1450
-	-1   0    0    1
-$EndComp
-$Comp
-L power:GND #PWR017
-U 1 1 60853DAC
-P 5100 1550
-F 0 "#PWR017" H 5100 1300 50  0001 C CNN
-F 1 "GND" H 5105 1377 50  0000 C CNN
-F 2 "" H 5100 1550 50  0001 C CNN
-F 3 "" H 5100 1550 50  0001 C CNN
-	1    5100 1550
-	1    0    0    -1
-$EndComp
-Wire Wire Line
-	5250 1550 5100 1550
-Text Label 5800 1450 0    50   ~ 0
+Text Label 3000 1050 0    50   ~ 0
 VIN_TPS
-Wire Wire Line
-	5650 1450 5800 1450
 Text Label 1050 1750 2    50   ~ 0
 VIN_TPS
 Wire Wire Line
 	1050 1750 1750 1750
+$Comp
+L EIPP_LIBRARY:EG1218 S?
+U 1 1 608ECEC4
+P 2600 1150
+AR Path="/60925CA4/60835FC2/608ECEC4" Ref="S?"  Part="1"
+AR Path="/60925CA4/6094117B/608ECEC4" Ref="S?"  Part="1"
+AR Path="/607D64D2/607D650A/608ECEC4" Ref="S9"  Part="1"
+F 0 "S9" H 2876 1196 50  0000 L CNN
+F 1 "EG1218" H 2876 1105 50  0000 L CNN
+F 2 "EIPP:EG1218" H 2600 1150 50  0001 L BNN
+F 3 "" H 2600 1150 50  0001 L BNN
+	1    2600 1150
+	0    -1   -1   0
+$EndComp
+Wire Wire Line
+	2800 1050 3000 1050
+Wire Wire Line
+	2200 1150 2200 1200
+Wire Wire Line
+	2400 1150 2200 1150
+$Comp
+L power:GND #PWR?
+U 1 1 608ECECD
+P 2200 1200
+AR Path="/607D64D2/607F1961/608ECECD" Ref="#PWR?"  Part="1"
+AR Path="/608CA2DC/608CBCF1/608ECECD" Ref="#PWR?"  Part="1"
+AR Path="/60925CA4/60926DAB/608ECECD" Ref="#PWR?"  Part="1"
+AR Path="/60925CA4/6094117B/608ECECD" Ref="#PWR?"  Part="1"
+AR Path="/60925CA4/60835FC2/608ECECD" Ref="#PWR?"  Part="1"
+AR Path="/607D64D2/607D650A/608ECECD" Ref="#PWR017"  Part="1"
+F 0 "#PWR017" H 2200 950 50  0001 C CNN
+F 1 "GND" H 2205 1027 50  0000 C CNN
+F 2 "" H 2200 1200 50  0001 C CNN
+F 3 "" H 2200 1200 50  0001 C CNN
+	1    2200 1200
+	1    0    0    -1
+$EndComp
+Wire Wire Line
+	2200 950  2400 950
+Wire Wire Line
+	2200 850  2200 950
+$Comp
+L power:+BATT #PWR?
+U 1 1 608ECED5
+P 2200 850
+AR Path="/607D64D2/607F1961/608ECED5" Ref="#PWR?"  Part="1"
+AR Path="/608CA2DC/608CBCF1/608ECED5" Ref="#PWR?"  Part="1"
+AR Path="/60925CA4/60926DAB/608ECED5" Ref="#PWR?"  Part="1"
+AR Path="/60925CA4/6094117B/608ECED5" Ref="#PWR?"  Part="1"
+AR Path="/60925CA4/60835FC2/608ECED5" Ref="#PWR?"  Part="1"
+AR Path="/607D64D2/607D650A/608ECED5" Ref="#PWR09"  Part="1"
+F 0 "#PWR09" H 2200 700 50  0001 C CNN
+F 1 "+BATT" H 2215 1023 50  0000 C CNN
+F 2 "" H 2200 850 50  0001 C CNN
+F 3 "" H 2200 850 50  0001 C CNN
+	1    2200 850
+	1    0    0    -1
+$EndComp
 $EndSCHEMATC
