File: file6086062F.sch (KiCad schematic (older format))
At the start: 13 parts, among them SW3 SW_SPDT, U4 ADP2302ARDZ

Commit message: full schematic, version 1.0
Parts:
- removed SW3: SW_SPDT, symbol Switch:SW_SPDT
- added S7: EG1218, EIPP:EG1218, symbol EIPP_LIBRARY:EG1218
- C17: footprint (none) -> Capacitor_SMD:C_0805_2012Metric_Pad1.18x1.45mm_HandSolder
- C18: footprint (none) -> Capacitor_SMD:C_0603_1608Metric_Pad1.08x0.95mm_HandSolder
- C19, C20: footprint (none) -> Capacitor_SMD:C_1206_3216Metric_Pad1.33x1.80mm_HandSolder
- D1: footprint (none) -> Diode_SMD:D_SOD-123
- L3: footprint (none) -> EIPP:IND_1255AY-4R7M=P3
- R10, R11, R12, R8, R9: footprint (none) -> Resistor_SMD:R_0805_2012Metric_Pad1.20x1.40mm_HandSolder
- U4: footprint (none) -> EIPP:SOIC127P600X175-9N
Connections:
- net +BATT: now also S7.S
- net GND: now also S7.O
- net VIN_ADP: now also S7.P
Changed lines of the file:
@@
 $Descr A4 11693 8268
 encoding utf-8
-Sheet 5 10
+Sheet 5 15
 Title ""
 Date ""
@@
 F 0 "C17" H 3642 3396 50  0000 L CNN
 F 1 "10uF" H 3642 3305 50  0000 L CNN
-F 2 "" H 3550 3350 50  0001 C CNN
+F 2 "Capacitor_SMD:C_0805_2012Metric_Pad1.18x1.45mm_HandSolder" H 3550 3350 50  0001 C CNN
 F 3 "~" H 3550 3350 50  0001 C CNN
 	1    3550 3350
@@
 	3550 3250 3550 3200
 Connection ~ 3550 3200
-$Comp
-L Switch:SW_SPDT SW3
-U 1 1 60863C95
-P 3500 2200
-F 0 "SW3" H 3500 1875 50  0000 C CNN
-F 1 "SW_SPDT" H 3500 1966 50  0000 C CNN
-F 2 "" H 3500 2200 50  0001 C CNN
-F 3 "~" H 3500 2200 50  0001 C CNN
-	1    3500 2200
-	-1   0    0    1
-$EndComp
-$Comp
-L power:GND #PWR019
-U 1 1 60864C54
-P 3150 2400
-F 0 "#PWR019" H 3150 2150 50  0001 C CNN
-F 1 "GND" H 3155 2227 50  0000 C CNN
-F 2 "" H 3150 2400 50  0001 C CNN
-F 3 "" H 3150 2400 50  0001 C CNN
-	1    3150 2400
-	1    0    0    -1
-$EndComp
-Wire Wire Line
-	3150 2400 3150 2300
-Wire Wire Line
-	3150 2300 3300 2300
-Wire Wire Line
-	3300 2100 3150 2100
-Wire Wire Line
-	3150 2100 3150 2000
-$Comp
-L power:+BATT #PWR018
-U 1 1 60865FB3
-P 3150 2000
-F 0 "#PWR018" H 3150 1850 50  0001 C CNN
-F 1 "+BATT" H 3165 2173 50  0000 C CNN
-F 2 "" H 3150 2000 50  0001 C CNN
-F 3 "" H 3150 2000 50  0001 C CNN
-	1    3150 2000
-	1    0    0    -1
-$EndComp
-Text Label 3800 2200 0    50   ~ 0
+Text Label 2250 2350 0    50   ~ 0
 VIN_ADP
-Wire Wire Line
-	3700 2200 3800 2200
 Text Label 3050 3200 2    50   ~ 0
 VIN_ADP
@@
 F 0 "U4" H 5125 3225 50  0000 C CNN
 F 1 "ADP2302ARDZ" H 5125 3134 50  0000 C CNN
-F 2 "" H 5150 3100 50  0001 C CNN
+F 2 "EIPP:SOIC127P600X175-9N" H 5150 3100 50  0001 C CNN
 F 3 "" H 5150 3100 50  0001 C CNN
 	1    5100 3100
@@
 F 0 "R12" H 6459 3746 50  0000 L CNN
 F 1 "10k2" H 6459 3655 50  0000 L CNN
-F 2 "" H 6400 3700 50  0001 C CNN
+F 2 "Resistor_SMD:R_0805_2012Metric_Pad1.20x1.40mm_HandSolder" H 6400 3700 50  0001 C CNN
 F 3 "~" H 6400 3700 50  0001 C CNN
 	1    6400 3700
@@
 F 0 "R11" H 6459 3346 50  0000 L CNN
 F 1 "31k6" H 6459 3255 50  0000 L CNN
-F 2 "" H 6400 3300 50  0001 C CNN
+F 2 "Resistor_SMD:R_0805_2012Metric_Pad1.20x1.40mm_HandSolder" H 6400 3300 50  0001 C CNN
 F 3 "~" H 6400 3300 50  0001 C CNN
 	1    6400 3300
@@
 F 0 "C20" H 7100 3400 50  0000 L CNN
 F 1 "47uF" H 7100 3200 50  0000 L CNN
-F 2 "" H 7100 3300 50  0001 C CNN
+F 2 "Capacitor_SMD:C_1206_3216Metric_Pad1.33x1.80mm_HandSolder" H 7100 3300 50  0001 C CNN
 F 3 "~" H 7100 3300 50  0001 C CNN
 	1    7100 3300
@@
 F 0 "D1" V 6096 2730 50  0000 R CNN
 F 1 "SSB43L" V 6005 2730 50  0000 R CNN
-F 2 "" V 6050 2800 50  0001 C CNN
+F 2 "Diode_SMD:D_SOD-123" V 6050 2800 50  0001 C CNN
 F 3 "~" V 6050 2800 50  0001 C CNN
 	1    6050 2800
@@
 F 0 "C18" V 5979 3200 50  0000 C CNN
 F 1 "0u1F" V 5888 3200 50  0000 C CNN
-F 2 "" H 5750 3200 50  0001 C CNN
+F 2 "Capacitor_SMD:C_0603_1608Metric_Pad1.08x0.95mm_HandSolder" H 5750 3200 50  0001 C CNN
 F 3 "~" H 5750 3200 50  0001 C CNN
 	1    5750 3200
@@
 F 0 "L3" V 6385 3100 50  0000 C CNN
 F 1 "4.7uH" V 6294 3100 50  0000 C CNN
-F 2 "" H 6200 3100 50  0001 C CNN
+F 2 "EIPP:IND_1255AY-4R7M=P3" H 6200 3100 50  0001 C CNN
 F 3 "~" H 6200 3100 50  0001 C CNN
 	1    6200 3100
@@
 F 0 "R10" V 4696 3350 50  0000 C CNN
 F 1 "100k" V 4605 3350 50  0000 C CNN
-F 2 "" H 4500 3350 50  0001 C CNN
+F 2 "Resistor_SMD:R_0805_2012Metric_Pad1.20x1.40mm_HandSolder" H 4500 3350 50  0001 C CNN
 F 3 "~" H 4500 3350 50  0001 C CNN
 	1    4500 3350
@@
 F 0 "R8" H 4059 3396 50  0000 L CNN
 F 1 "56k" H 4059 3305 50  0000 L CNN
-F 2 "" H 4000 3350 50  0001 C CNN
+F 2 "Resistor_SMD:R_0805_2012Metric_Pad1.20x1.40mm_HandSolder" H 4000 3350 50  0001 C CNN
 F 3 "~" H 4000 3350 50  0001 C CNN
 	1    4000 3350
@@
 F 0 "R9" H 4059 3796 50  0000 L CNN
 F 1 "10k2" H 4059 3705 50  0000 L CNN
-F 2 "" H 4000 3750 50  0001 C CNN
+F 2 "Resistor_SMD:R_0805_2012Metric_Pad1.20x1.40mm_HandSolder" H 4000 3750 50  0001 C CNN
 F 3 "~" H 4000 3750 50  0001 C CNN
 	1    4000 3750
@@
 F 0 "C19" H 6800 3400 50  0000 L CNN
 F 1 "47uF" H 6800 3200 50  0000 L CNN
-F 2 "" H 6800 3300 50  0001 C CNN
+F 2 "Capacitor_SMD:C_1206_3216Metric_Pad1.33x1.80mm_HandSolder" H 6800 3300 50  0001 C CNN
 F 3 "~" H 6800 3300 50  0001 C CNN
 	1    6800 3300
@@
 Wire Wire Line
 	6800 3450 6800 3400
+$Comp
+L EIPP_LIBRARY:EG1218 S?
+U 1 1 608E4B60
+P 1750 2450
+AR Path="/60925CA4/60835FC2/608E4B60" Ref="S?"  Part="1"
+AR Path="/60925CA4/6094117B/608E4B60" Ref="S?"  Part="1"
+AR Path="/607D64D2/60860630/608E4B60" Ref="S7"  Part="1"
+F 0 "S7" H 2026 2496 50  0000 L CNN
+F 1 "EG1218" H 2026 2405 50  0000 L CNN
+F 2 "EIPP:EG1218" H 1750 2450 50  0001 L BNN
+F 3 "" H 1750 2450 50  0001 L BNN
+	1    1750 2450
+	0    -1   -1   0
+$EndComp
+Wire Wire Line
+	1350 2450 1350 2500
+Wire Wire Line
+	1550 2450 1350 2450
+$Comp
+L power:GND #PWR?
+U 1 1 608E4B69
+P 1350 2500
+AR Path="/607D64D2/607F1961/608E4B69" Ref="#PWR?"  Part="1"
+AR Path="/608CA2DC/608CBCF1/608E4B69" Ref="#PWR?"  Part="1"
+AR Path="/60925CA4/60926DAB/608E4B69" Ref="#PWR?"  Part="1"
+AR Path="/60925CA4/6094117B/608E4B69" Ref="#PWR?"  Part="1"
+AR Path="/60925CA4/60835FC2/608E4B69" Ref="#PWR?"  Part="1"
+AR Path="/607D64D2/60860630/608E4B69" Ref="#PWR019"  Part="1"
+F 0 "#PWR019" H 1350 2250 50  0001 C CNN
+F 1 "GND" H 1355 2327 50  0000 C CNN
+F 2 "" H 1350 2500 50  0001 C CNN
+F 3 "" H 1350 2500 50  0001 C CNN
+	1    1350 2500
+	1    0    0    -1
+$EndComp
+Wire Wire Line
+	1350 2250 1550 2250
+Wire Wire Line
+	1350 2150 1350 2250
+$Comp
+L power:+BATT #PWR?
+U 1 1 608E4B71
+P 1350 2150
+AR Path="/607D64D2/607F1961/608E4B71" Ref="#PWR?"  Part="1"
+AR Path="/608CA2DC/608CBCF1/608E4B71" Ref="#PWR?"  Part="1"
+AR Path="/60925CA4/60926DAB/608E4B71" Ref="#PWR?"  Part="1"
+AR Path="/60925CA4/6094117B/608E4B71" Ref="#PWR?"  Part="1"
+AR Path="/60925CA4/60835FC2/608E4B71" Ref="#PWR?"  Part="1"
+AR Path="/607D64D2/60860630/608E4B71" Ref="#PWR018"  Part="1"
+F 0 "#PWR018" H 1350 2000 50  0001 C CNN
+F 1 "+BATT" H 1365 2323 50  0000 C CNN
+F 2 "" H 1350 2150 50  0001 C CNN
+F 3 "" H 1350 2150 50  0001 C CNN
+	1    1350 2150
+	1    0    0    -1
+$EndComp
+Wire Wire Line
+	1950 2350 2250 2350
 $EndSCHEMATC
