File: file608DA413.sch (KiCad schematic (older format))
At the start: 0 parts

Commit message: full schematic, version 1.0
Parts:
- added C27: 10uF, Capacitor_SMD:C_0805_2012Metric_Pad1.18x1.45mm_HandSolder, symbol Device:C_Small
- added C28: 100nF, Capacitor_SMD:C_0603_1608Metric_Pad1.08x0.95mm_HandSolder, symbol Device:C_Small
- added C29, C30, C31: 47uF, Capacitor_SMD:C_1206_3216Metric_Pad1.33x1.80mm_HandSolder, symbol Device:C_Small
- added L5: 4.7uH, EIPP:IND_1255AY-4R7M=P3, symbol Device:L_Small
- added R22: 56k, Resistor_SMD:R_0603_1608Metric_Pad0.98x0.95mm_HandSolder, symbol Device:R_Small
- added R23: 10k, Resistor_SMD:R_0805_2012Metric_Pad1.20x1.40mm_HandSolder, symbol Device:R_Small
- added R44: 700R, Resistor_SMD:R_0603_1608Metric_Pad0.98x0.95mm_HandSolder, symbol Device:R_Small
- added S5: EG1218, EIPP:EG1218, symbol EIPP_LIBRARY:EG1218
- added U7: TPS563231DRLR, EIPP:SOT50P160X60-6N, symbol EIPP_LIBRARY:TPS563231DRLR
Connections:
- new net: R22.2, R44.1
- new net: R44.2, U7.6 (FB)
- new net: C28.1, L5.1, U7.2 (SW)
- new net: C28.2, U7.4 (BST)
- new net +BATT: S5.S
- new net GND: C27.2, C29.2, C30.2, C31.2, R23.2, S5.O, U7.3 (GND)
- new net TPS_4V: C29.1, C30.1, C31.1, L5.2, R22.1, R23.1
- new net VIN_TPS: C27.1, S5.P, U7.1 (VIN), U7.5 (EN)
