File: PWR_SUB_SYS_PCB.kicad_pcb (KiCad board)
At the start: 2 copper layers, 98 x 100 mm, 147 parts, among them J1 Conn_01x06_Female, U1 TPS54228DDA, U10 LM2731YMF, U11 TPS61175PWP, U2 MP2235, U3 INA4180A1IPWR, U4 ADP2302ARDZ, U5 254, U6 MP2235, U7 TPS563231DRLR, U8 TPS563207DRLR, U9 LMR62014XMFE_NOPB

Commit message: incomplete pcb
Parts:
- C1, C10, C11, C2, C3, C32, C33, C34, C35, C36, C37, C4, C41, C43, C44, C5, C8, C9, D3, L1, L6, L8, R1, R2, R24, R25, R26, R27, R3, R30, R35, R36, R37, R38, R39, R40, R45, R47, U1, U10, U8: moved to F.Cu
- moved C10 142.6 mm to (42.8, 92.9)
- moved C11 141.3 mm to (42.8, 95.6)
- moved R3 141.2 mm to (33.3, 95.9), turned to 90 degrees
- moved C8 140.5 mm to (26.9, 97.4), turned to 90 degrees
- moved R1 140.5 mm to (29.5, 97.4), turned to 90 degrees
- moved C1 140.4 mm to (42.1, 97.9)
- moved R2 139.4 mm to (28.6, 100.6)
- moved U1 139.2 mm to (36.1, 101.2)
- moved C4 139.2 mm to (41.7, 101.3), turned to 90 degrees
- moved C2 139.0 mm to (29.6, 102.2)
- moved L1 138.9 mm to (49.7, 102.6), turned to 90 degrees
- moved C3 138.2 mm to (33.4, 105.9), turned to 270 degrees
- moved C5 138.1 mm to (48.6, 106.9)
- moved S9 137.9 mm to (37.0, 113.3)
- moved C9 137.9 mm to (48.6, 109.3)
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Connections:
- U1 pad 10: (no net) -> GND
- U1 pad 11: (no net) -> GND
- U1 pad 12: (no net) -> GND
- U1 pad 13: (no net) -> GND
- U1 pad 14: (no net) -> GND
- U1 pad 15: (no net) -> GND
- U1 pad 16: (no net) -> GND
- U1 pad 17: (no net) -> GND
- U11 pad 16: (no net) -> GND
- U11 pad 17: (no net) -> GND
- U11 pad 18: (no net) -> GND
- U11 pad 19: (no net) -> GND
- U11 pad 20: (no net) -> GND
- U11 pad 21: (no net) -> GND
Routing:
- net +BATT: track 0.00 -> 245.1 mm, vias 0 -> 2
- net 3V3: track 0.00 -> 81.2 mm, vias 0 -> 2
- net 12V_TPS: track 0.00 -> 72.4 mm, vias 0 -> 1
- net LOAD_1: track 0.00 -> 72.3 mm, vias 0 -> 5
- net 12V_LM27: track 0.00 -> 61.2 mm, vias 0 -> 3
- net 12V: track 0.00 -> 59.9 mm, vias 0 -> 2
- net 12V_LMR52: track 0.00 -> 40.4 mm, vias 0 -> 1
- net LOAD_3: track 0.00 -> 38.8 mm
- net GND: track 0.00 -> 27.5 mm
- net /12V/LMR52014/VIN_LMR: track 0.00 -> 26.3 mm, vias 0 -> 1
- net TPS_4V: track 0.00 -> 25.3 mm, vias 0 -> 2
- net /12V/TPS61175PWP/VIN_TPS: track 0.00 -> 24.1 mm
- net /12V/LM2731YMF/VIN_LMR: track 0.00 -> 22.4 mm
- net /4V/MP2235_4V/VIN_MP: track 0.00 -> 21.5 mm
- net /4V/TPS563231/VIN_TPS: track 0.00 -> 21.1 mm
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Other:
- net class Default: clearance 0.2 -> 0.1
- rule trace_clearance: 0.2 -> 0.1

Commit message: finished pcb v1
Parts:
- C17, C18, C19, C20, D1, L3, R10, R11, R12, R8, R9, U4: moved to B.Cu
- J1: footprint Connector_PinHeader_2.54mm:PinHeader_1x06_P2.54mm_Vertical -> Connector_PinSocket_2.54mm:PinSocket_1x06_P2.54mm_Vertical
- R41, R42, R43: moved to F.Cu
- moved S9 170.5 mm to (207.3, 103.5)
- moved R8 161.7 mm to (216.1, 111.9)
- moved R9 161.7 mm to (220.0, 112.1)
- moved R10 161.6 mm to (212.6, 112.3), turned to 270 degrees
- moved R12 161.4 mm to (225.0, 113.0)
- moved C17 160.5 mm to (210.9, 116.4), turned to 90 degrees
- moved R11 160.5 mm to (224.0, 116.6), turned to 90 degrees
- moved U4 160.5 mm to (217.3, 116.8)
- moved C18 159.8 mm to (213.7, 121.5), turned to 270 degrees
- moved D1 159.8 mm to (218.1, 121.8)
- moved C20 159.8 mm to (226.7, 122.1)
- moved L3 159.8 mm to (218.4, 126.6)
- moved C19 159.7 mm to (226.5, 124.9)
- moved C8 154.1 mm to (180.8, 105.2)
- moved R1 154.1 mm to (183.4, 105.2)
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Connections:
- A1 pad 22: /Data logging/A3 -> Net-(A1-Pad22)
- U3 pad 14: /Data logging/A3 -> Net-(U3-Pad14)
Routing:
- net +BATT: track 245.1 -> 367.3 mm, vias 2 -> 8
- net GND: track 27.5 -> 139.6 mm, vias 0 -> 14
- net /Data logging/SS: track 0.00 -> 90.3 mm, vias 0 -> 2
- net /Data logging/5V: track 2.44 -> 90.4 mm, vias 0 -> 5
- net MP_4V: track 11.1 -> 92.2 mm, vias 0 -> 4
- net /Data logging/MOSI: track 0.00 -> 80.4 mm, vias 0 -> 2
- net /Data logging/A0: track 0.00 -> 78.5 mm, vias 0 -> 6
- net TPS2_4V: track 0.00 -> 78.2 mm, vias 0 -> 2
- net /Data logging/A2: track 0.00 -> 71.8 mm, vias 0 -> 6
- net /Data logging/MISO: track 0.00 -> 70.6 mm
- net ADP_3V3: track 5.63 -> 74.8 mm, vias 0 -> 2
- net MP_3V3: track 5.57 -> 74.6 mm, vias 0 -> 4
- net /Data logging/A1: track 0.00 -> 65.4 mm, vias 0 -> 2
- net /Data logging/SCK: track 0.00 -> 64.0 mm
- net 4V: track 6.94 -> 63.1 mm, vias 0 -> 3
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- added copper zone on B.Cu, net GND
- added copper zone on F.Cu, net GND

Commit message: finished pcb v2
Parts:
- removed C42, C45, C46: 4.7uF, Capacitor_SMD:C_1206_3216Metric_Pad1.33x1.80mm_HandSolder
- removed C47: 10uF, Capacitor_SMD:C_0805_2012Metric_Pad1.18x1.45mm_HandSolder
- removed C48: 47nF, Capacitor_SMD:C_0805_2012Metric_Pad1.18x1.45mm_HandSolder
- removed C49: 33nF, Capacitor_SMD:C_0805_2012Metric_Pad1.18x1.45mm_HandSolder
- removed D4: D_Schottky, Diode_SMD:D_SOD-123
- removed L9: 12uH, EIPP:SDR0805
- removed R32: 16.2k, Resistor_SMD:R_0805_2012Metric_Pad1.20x1.40mm_HandSolder
- removed R33: 86.6k, Resistor_SMD:R_0805_2012Metric_Pad1.20x1.40mm_HandSolder
- removed R34: 2.32k, Resistor_SMD:R_0805_2012Metric_Pad1.20x1.40mm_HandSolder
- removed S1: EG1218, EIPP:EG1218
- removed U11: TPS61175PWP, EIPP:IC_TPS27S100BPWPR
- added C50: 22uF, Capacitor_SMD:C_1210_3225Metric_Pad1.33x2.70mm_HandSolder, F.Cu at (214.5, 139.1)
- added C51: 1uF, Capacitor_SMD:C_0805_2012Metric_Pad1.18x1.45mm_HandSolder, F.Cu at (202.3, 140.0)
- added C52: 680p, Capacitor_SMD:C_0603_1608Metric_Pad1.08x0.95mm_HandSolder, F.Cu at (212.1, 145.8)
- added C53: 390nF, Capacitor_SMD:C_0603_1608Metric_Pad1.08x0.95mm_HandSolder, F.Cu at (213.9, 145.8)
- added C54: 4.7nF, Capacitor_SMD:C_0805_2012Metric, F.Cu at (214.6, 149.7)
- added C55: 47uF, Capacitor_THT:CP_Radial_D5.0mm_P2.00mm, F.Cu at (200.4, 152.8)
- added C56: 47uF, Capacitor_THT:CP_Radial_D5.0mm_P2.00mm, F.Cu at (194.5, 152.8)
- added C57: 47uF, Capacitor_THT:CP_Radial_D5.0mm_P2.00mm, F.Cu at (206.2, 152.7)
- added D14: STPS1L20M, EIPP:STPS1L20M, F.Cu at (202.0, 141.9)
- added D15: STPS1L20M, EIPP:STPS1L20M, F.Cu at (213.9, 158.7)
- added L10: 27 uH, EIPP:744770127, F.Cu at (220.2, 139.8)
- added Q1: STN4NF03L, EIPP:STN4NF03L, F.Cu at (225.8, 151.0)
- added R48: 0R1, Resistor_SMD:R_1020_2550Metric_Pad1.33x5.20mm_HandSolder, F.Cu at (149.3, 96.3)
- added R50: 1k8, Resistor_SMD:R_0805_2012Metric_Pad1.20x1.40mm_HandSolder, F.Cu at (214.6, 143.0)
- added R51: 2k2, Resistor_SMD:R_0805_2012Metric_Pad1.20x1.40mm_HandSolder, F.Cu at (211.7, 148.8)
- added R52: 82k, Resistor_SMD:R_0805_2012Metric_Pad1.20x1.40mm_HandSolder, F.Cu at (216.9, 149.8)
- added R53: 4k32, Resistor_SMD:R_0805_2012Metric_Pad1.20x1.40mm_HandSolder, F.Cu at (216.5, 145.9)
- added S13: EG1218, EIPP:EG1218, F.Cu at (205.8, 136.4)
- added U12: L7981A-Regulator_Switching, EIPP:L7981A, F.Cu at (207.0, 144.3)
- R31: value 143k -> 1k
- moved R31 20.7 mm to (203.0, 144.3), turned to 90 degrees
- moved BT4 4.52 mm to (143.0, 93.2)
- moved BT1 2.29 mm to (140.4, 80.6)
- moved BT3 1.94 mm to (140.5, 89.1)
- moved BT2 0.68 mm to (143.1, 84.6)
Connections:
- A1 pad 22: Net-(A1-Pad22) -> /Data logging/A3
- BT1 pad 1: +BATT -> VCC
- BT2 pad 2: GND -> +8V
- BT3 pad 1: +BATT -> VCC
- BT4 pad 2: GND -> +8V
- R31 pad 1: 12V_TPS -> Net-(R31-Pad1)
- R31 pad 2: Net-(R31-Pad2) -> /12V/L7981A/VIN_L798
- R37 pad 1: 12V_TPS -> 12V_L7891A
- S10 pad 4: 12V_TPS -> 12V_L7891A
- U3 pad 12: Net-(U3-Pad12) -> +8V
- U3 pad 13: Net-(U3-Pad13) -> +BATT
- U3 pad 14: Net-(U3-Pad14) -> /Data logging/A3
Routing:
- net /Data logging/A3: track 0.00 -> 113.7 mm, vias 0 -> 5
- net 12V_TPS: track 79.5 -> 0.00 mm, vias 1 -> 0
- net 12V_L7891A: track 0.00 -> 72.7 mm
- net +8V: track 0.00 -> 56.7 mm, vias 0 -> 2
- net Net-(D14-Pad1): track 0.00 -> 33.7 mm, vias 0 -> 2
- net +BATT: track 367.3 -> 336.8 mm
- net Net-(D15-Pad2): track 0.00 -> 27.7 mm
- net /12V/TPS61175PWP/VIN_TPS: track 24.1 -> 0.00 mm
- net Net-(C52-Pad1): track 0.00 -> 22.0 mm, vias 0 -> 3
- net GND: track 139.6 -> 160.4 mm, vias 14 -> 24
- net /12V/L7981A/VIN_L798: track 0.00 -> 19.0 mm
- net Net-(D4-Pad2): track 16.5 -> 0.00 mm, vias 2 -> 0
- net Net-(R31-Pad1): track 0.00 -> 13.5 mm, vias 0 -> 2
- net VCC: track 0.00 -> 10.0 mm
- net Net-(R33-Pad1): track 7.83 -> 0.00 mm, vias 2 -> 0
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Other:
- board text added: "12 V L7981A"
- board text removed: "12 V TPS"
