File: file6080506E.sch (KiCad schematic (older format))
At the start: 4 parts

Commit message: full schematic, version 1.0
Parts:
- BT1, BT2, BT3, BT4: footprint (none) -> Connector_PinHeader_2.54mm:PinHeader_1x02_P2.54mm_Vertical
Changed lines of the file:
@@
 $Descr A4 11693 8268
 encoding utf-8
-Sheet 7 10
+Sheet 7 15
 Title ""
 Date ""
@@
 F 0 "BT1" H 2868 2796 50  0000 L CNN
 F 1 "Battery_Cell" H 2868 2705 50  0000 L CNN
-F 2 "" V 2750 2760 50  0001 C CNN
+F 2 "Connector_PinHeader_2.54mm:PinHeader_1x02_P2.54mm_Vertical" V 2750 2760 50  0001 C CNN
 F 3 "~" V 2750 2760 50  0001 C CNN
 	1    2750 2700
@@
 F 0 "BT3" H 3168 2796 50  0000 L CNN
 F 1 "Battery_Cell" H 3168 2705 50  0000 L CNN
-F 2 "" V 3050 2760 50  0001 C CNN
+F 2 "Connector_PinHeader_2.54mm:PinHeader_1x02_P2.54mm_Vertical" V 3050 2760 50  0001 C CNN
 F 3 "~" V 3050 2760 50  0001 C CNN
 	1    3050 2700
@@
 F 0 "BT2" H 2868 3196 50  0000 L CNN
 F 1 "Battery_Cell" H 2868 3105 50  0000 L CNN
-F 2 "" V 2750 3160 50  0001 C CNN
+F 2 "Connector_PinHeader_2.54mm:PinHeader_1x02_P2.54mm_Vertical" V 2750 3160 50  0001 C CNN
 F 3 "~" V 2750 3160 50  0001 C CNN
 	1    2750 3100
@@
 F 0 "BT4" H 3168 3196 50  0000 L CNN
 F 1 "Battery_Cell" H 3168 3105 50  0000 L CNN
-F 2 "" V 3050 3160 50  0001 C CNN
+F 2 "Connector_PinHeader_2.54mm:PinHeader_1x02_P2.54mm_Vertical" V 3050 3160 50  0001 C CNN
 F 3 "~" V 3050 3160 50  0001 C CNN
 	1    3050 3100

Commit message: finished pcb v2
Connections:
- net labels added: +8V, VCC
- net labels removed: +BATT, GND
Changed lines of the file:
@@
 Wire Wire Line
 	2900 2350 3050 2350
-$Comp
-L power:+BATT #PWR027
-U 1 1 60807E66
-P 2900 2100
-F 0 "#PWR027" H 2900 1950 50  0001 C CNN
-F 1 "+BATT" H 2915 2273 50  0000 C CNN
-F 2 "" H 2900 2100 50  0001 C CNN
-F 3 "" H 2900 2100 50  0001 C CNN
-	1    2900 2100
-	1    0    0    -1
-$EndComp
 Wire Wire Line
 	2900 3400 2900 3650
@@
 Wire Wire Line
 	2900 3400 3050 3400
-$Comp
-L power:GND #PWR028
-U 1 1 608087E1
-P 2900 3650
-F 0 "#PWR028" H 2900 3400 50  0001 C CNN
-F 1 "GND" H 2905 3477 50  0000 C CNN
-F 2 "" H 2900 3650 50  0001 C CNN
-F 3 "" H 2900 3650 50  0001 C CNN
-	1    2900 3650
-	1    0    0    -1
-$EndComp
 $Comp
 L power:PWR_FLAG #FLG0101
@@
 Wire Wire Line
 	2600 2250 2900 2250
-Connection ~ 2900 2250
-Wire Wire Line
-	2900 2250 2900 2100
 $Comp
 L power:PWR_FLAG #FLG0102
@@
 Wire Wire Line
 	2450 3400 2750 3400
+Connection ~ 2900 2250
+Wire Wire Line
+	2900 2250 2900 2100
+$Comp
+L power:VCC #PWR0116
+U 1 1 609DD988
+P 2900 2100
+F 0 "#PWR0116" H 2900 1950 50  0001 C CNN
+F 1 "VCC" H 2915 2273 50  0000 C CNN
+F 2 "" H 2900 2100 50  0001 C CNN
+F 3 "" H 2900 2100 50  0001 C CNN
+	1    2900 2100
+	1    0    0    -1
+$EndComp
+$Comp
+L power:+8V #PWR0117
+U 1 1 609DFFCC
+P 2900 3650
+F 0 "#PWR0117" H 2900 3500 50  0001 C CNN
+F 1 "+8V" V 2915 3778 50  0000 L CNN
+F 2 "" H 2900 3650 50  0001 C CNN
+F 3 "" H 2900 3650 50  0001 C CNN
+	1    2900 3650
+	0    -1   -1   0
+$EndComp
 $EndSCHEMATC
